File: sensor-board/sensor-board.kicad_pcb (KiCad board)
At the start: 2 copper layers, 35.6 x 33 mm, 28 parts, among them U1 CE_HEADER, U2 74HC595, U3 DS7505

Commit message: Finishing off Teensy project
Parts:
- C1, C2, R1, R10, R11, R12, R14, R15, R2, R3, R4, R5, R6, R7, R8, R9, U1: moved to B.Cu
- moved U2 54.3 mm to (89.5, 99.9)
- moved R12 52.6 mm to (89.4, 113.3), turned to 0 degrees
- moved C1 50.5 mm to (86.9, 98.0), turned to 90 degrees
- moved R1 49.9 mm to (98.6, 96.0), turned to 180 degrees
- moved R2 49.6 mm to (98.6, 99.1), turned to 180 degrees
- moved R3 49.2 mm to (98.6, 102.1), turned to 180 degrees
- moved R4 49.0 mm to (98.6, 105.2), turned to 180 degrees
- moved R5 48.7 mm to (98.6, 108.2), turned to 180 degrees
- moved C2 48.7 mm to (89.4, 101.5)
- moved R6 48.4 mm to (98.6, 111.3), turned to 180 degrees
- moved R7 48.2 mm to (98.6, 114.3), turned to 180 degrees
- moved R8 47.9 mm to (98.6, 117.3), turned to 180 degrees
- moved D1 46.9 mm to (98.6, 96.0)
- moved D2 46.6 mm to (98.6, 99.1)
- moved D3 46.3 mm to (98.6, 102.1)
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Routing:
- net GND: track 22.8 -> 85.8 mm, vias 17 -> 3
- net +3V3: track 0.00 -> 46.9 mm, vias 0 -> 4
- net /PR_BOT: track 67.6 -> 29.7 mm
- net /PR_TOP: track 73.5 -> 35.8 mm
- net /dataPin: track 29.4 -> 17.4 mm, vias 1 -> 0
- net Net-(D8-Pad2): track 10.6 -> 20.1 mm
- net /latchPin: track 29.7 -> 22.0 mm
- net Net-(D7-Pad2): track 5.53 -> 12.8 mm
- net Net-(D1-Pad2): track 12.6 -> 6.06 mm
- net Net-(D6-Pad2): track 6.05 -> 12.3 mm
- net Net-(D2-Pad2): track 11.3 -> 6.17 mm
- net /clockPin: track 25.7 -> 20.7 mm, vias 1 -> 0
- net /SCL: track 14.6 -> 19.6 mm, vias 0 -> 2
- net Net-(D5-Pad2): track 7.20 -> 10.4 mm
- net Net-(D3-Pad2): track 10.0 -> 6.90 mm
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- removed copper zone on F.Cu, net +3V3
- removed copper zone on B.Cu, net GND
Other:
- board size 35.6 x 33 mm -> 25.4 x 25.4 mm
- board text added: "CE Sensor Board"
